Commit message: feeding deployment state

File: arms/gen3/6dof/urdf/gen3_macro.xacro (robot description, xacro)
@@ -11,5 +11,5 @@
       </inertial>
       <visual>
-        <origin xyz="0 0 0" rpy="0 0 -1.5708" />
+        <origin xyz="0 0 0" rpy="0 0 0" />
         <geometry>
           <mesh filename="package://kortex_description/arms/gen3/${dof}dof/meshes/base_link.STL" />
@@ -20,5 +20,5 @@
       </visual>
       <collision>
-        <origin xyz="0 0 0" rpy="0 0 -1.5708" />
+        <origin xyz="0 0 0" rpy="0 0 0" />
         <geometry>
           <mesh filename="package://kortex_description/arms/gen3/${dof}dof/meshes/base_link.STL" />
@@ -49,5 +49,5 @@
     </link>
     <joint name="${prefix}joint_1" type="continuous">
-      <origin xyz="0 0 0.15643" rpy="-3.1416 0.0 -1.5708" />
+      <origin xyz="0 0 0.15643" rpy="-3.1416 0.0 0" />
       <parent link="${prefix}base_link" />
       <child link="${prefix}shoulder_link" />
@@ -244,5 +244,5 @@
         xyz="0 0 0" />
     </joint>
-    <xacro:if value="${vision}">
+<!--     <xacro:if value="${vision}">
     <link name="${prefix}camera_link">
       <inertial>
@@ -283,5 +283,5 @@
       <axis xyz="0.001 0.001 0.001" />
     </joint>
-    </xacro:if>
+    </xacro:if> -->
   </xacro:macro>
 </robot>

File: arms/gen3/7dof/urdf/gen3_macro.xacro (robot description, xacro)
@@ -298,5 +298,11 @@
         velocity="1.2218" />
     </joint>
-    <link name="${prefix}end_effector_link" />
+    <link name="${prefix}end_effector_link">
+      <inertial>
+        <origin xyz="0 0 0" rpy="0 0 0" />
+        <mass value="0" />
+        <inertia ixx="0" ixy="0" ixz="0" iyy="0" iyz="0" izz="0" />
+      </inertial>
+    </link>
     <joint
       name="${prefix}end_effector"
@@ -311,5 +317,11 @@
     </joint>
     <xacro:if value="${vision}">
-      <link name="${prefix}camera_link" />
+      <link name="${prefix}camera_link">
+        <inertial>
+          <origin rpy="0 0 3.14" xyz="0.026 0.063 0.031" />
+          <mass value="0" />
+          <inertia ixx="0" ixy="0" ixz="0" iyy="0" iyz="0" izz="0" />
+        </inertial>
+      </link>
       <joint name="${prefix}camera_module" type="fixed">
         <origin xyz="0 0.05639 -0.00305" rpy="3.14159265358979 3.14159265358979 0" />
@@ -317,5 +329,11 @@
         <child  link="${prefix}camera_link" />
       </joint>
-      <link name="${prefix}camera_depth_frame" />
+      <link name="${prefix}camera_depth_frame">
+        <inertial>
+          <origin xyz="0 0 0" rpy="0 0 0" />
+          <mass value="0" />
+          <inertia ixx="0" ixy="0" ixz="0" iyy="0" iyz="0" izz="0" />
+        </inertial>
+      </link>
       <joint name="${prefix}depth_module" type="fixed">
         <origin xyz="0.0275 0.066 -0.00305" rpy="3.14159265358979 3.14159265358979 0" />
@@ -323,5 +341,11 @@
         <child  link="${prefix}camera_depth_frame" />
       </joint>
-      <link name="${prefix}camera_color_frame" />
+      <link name="${prefix}camera_color_frame">
+        <inertial>
+          <origin xyz="0 0 0" rpy="0 0 0" />
+          <mass value="0" />
+          <inertia ixx="0" ixy="0" ixz="0" iyy="0" iyz="0" izz="0" />
+        </inertial>
+      </link>
       <joint name="${prefix}color_module" type="fixed">
         <origin xyz="0 0.05639 -0.00305" rpy="3.14159265358979 3.14159265358979 0" />

File: grippers/robotiq_2f_85/urdf/robotiq_arg2f.xacro (robot description, xacro)
@@ -23,6 +23,6 @@
         <geometry>
           <!-- The DAE file doesn't show well in Gazebo so we're using the STL instead -->
-          <!-- <mesh filename="package://kortex_description/grippers/robotiq_2f_85/meshes/visual/robotiq_arg2f_85_base_link.dae" scale="0.001 0.001 0.001"/> -->
-          <mesh filename="package://kortex_description/grippers/robotiq_2f_85/meshes/collision/robotiq_arg2f_base_link.stl" />
+          <mesh filename="package://kortex_description/grippers/robotiq_2f_85/meshes/visual/robotiq_arg2f_85_base_link_realsense2.dae" scale="0.001 0.001 0.001"/>
+          <!-- <mesh filename="package://kortex_description/grippers/robotiq_2f_85/meshes/collision/robotiq_arg2f_base_link.stl" /> -->
         </geometry>
         <material name="">
@@ -45,8 +45,21 @@
         <inertial>
             <origin xyz="0 0 0.058" rpy="0 0 0"/>
-            <mass value="0.925"/>
+            <mass value="0.97"/>
             <inertia ixx="0.000000" ixy="0.000000" ixz="0.000000" iyy="0.000000" iyz="0.000000" izz="0.000000"/>
         </inertial>
     </link>
+    <link name="${prefix}finger_tip">
+      <inertial>
+        <origin xyz="0 0 0" rpy="0 0 0" />
+        <mass value="0" />
+        <inertia ixx="0" ixy="0" ixz="0" iyy="0" iyz="0" izz="0" />
+      </inertial>
+    </link>
+    <joint name="${prefix}finger_tip_joint" type="fixed">
+        <parent link="${parent}" />
+        <child link="${prefix}finger_tip" />
+        <origin xyz="0 0 0.163" rpy="0 0 0"/>
+        <!-- <axis xyz="0 0 1" /> -->
+    </joint>
     <gazebo reference="${prefix}robotiq_arg2f_base_link">
       <material>Gazebo/Black</material>

File: robots/gen3.xacro (robot description, xacro)
@@ -7,6 +7,7 @@
     <xacro:arg name="gripper" default="" />
     <xacro:arg name="sim" default="false" />
+    <xacro:arg name="feeding_utensil" default="false" />
     <xacro:arg name="prefix" default="" />
     <xacro:include filename="$(find kortex_description)/robots/kortex_robot.xacro" />
-    <xacro:load_robot arm="$(arg arm)" gripper="$(arg gripper)" dof="$(arg dof)" vision="$(arg vision)" sim="$(arg sim)" prefix="$(arg prefix)" />
+    <xacro:load_robot arm="$(arg arm)" gripper="$(arg gripper)" dof="$(arg dof)" vision="$(arg vision)" sim="$(arg sim)" feeding_utensil="$(arg feeding_utensil)" prefix="$(arg prefix)" />
 </robot>

File: robots/gen3_6dof_vision_forque.urdf (robot description, URDF)
Before this commit: robot gen3_robotiq_2f_85, 27 links, 26 joints
Links:
- removed link camera_link
- removed link depth_camera_link
- added link inline_forque_end_effector, mass 0
- link inertia_link: mass 0.925 -> 0.97
- link world: mass None -> 0
Joints:
- removed joint camera_color_joint
- removed joint camera_depth_joint
- added joint joint_inline_forque_end_effector: type fixed, parent forque, child inline_forque_end_effector, origin xyz=0 0 0.175 rpy=0 0 0, axis 0 0 0, limit lower=0 upper=0 effort=2000 velocity=1
- joint forque_joint: origin xyz=0.0 0.0 0.11 rpy=0.0 0.0 0 -> xyz=0.0 0.0 0.125 rpy=0.0 0.0 0
- joint joint_forque_end_effector: origin xyz=0 0.007 0.18 rpy=0 0 0 -> xyz=0 0 0.22 rpy=0 0 0
- joint joint_forque_tip: origin xyz=0.0 0.007 0.18 rpy=-0.5 0 0 -> xyz=0.0 0.007 0.175 rpy=-0.261799 0 0

File: robots/gen3_robotiq_2f_85.xacro (robot description, xacro)
@@ -6,10 +6,10 @@
     <xacro:arg name="vision" default="true" />
     <xacro:arg name="gripper" default="robotiq_2f_85" />
-    <xacro:arg name="forque" default="true" />
-    <xacro:arg name="realsense_cam" default="true" />
-    <xacro:arg name="reflect_cam" default="true" />
+    <xacro:arg name="forque" default="false" />
     <xacro:arg name="sim" default="false" />
     <xacro:arg name="prefix" default="" />
+    <xacro:arg name="feeding_utensil" default="false" />
+    <xacro:arg name="drinking_utensil" default="false" />
     <xacro:include filename="$(find kortex_description)/robots/kortex_robot.xacro" />
-    <xacro:load_robot arm="$(arg arm)" gripper="$(arg gripper)" forque="$(arg forque)" reflect_cam="$(arg reflect_cam)" realsense_cam="$(arg realsense_cam)" dof="$(arg dof)" vision="$(arg vision)" sim="$(arg sim)" prefix="$(arg prefix)" />
+    <xacro:load_robot arm="$(arg arm)" gripper="$(arg gripper)" forque="$(arg forque)" feeding_utensil="$(arg feeding_utensil)" drinking_utensil="$(arg drinking_utensil)"  dof="$(arg dof)" vision="$(arg vision)" sim="$(arg sim)" prefix="$(arg prefix)" />
 </robot>

File: robots/kortex_robot.xacro (robot description, xacro)
@@ -1,5 +1,5 @@
 <?xml version="1.0"?>
 <robot xmlns:xacro="http://ros.org/wiki/xacro">
-    <xacro:macro name="load_robot" params="arm gripper forque reflect_cam realsense_cam dof vision sim prefix">
+    <xacro:macro name="load_robot" params="arm gripper forque feeding_utensil drinking_utensil dof vision sim prefix">
         <!-- Files to include -->
         <xacro:include filename="$(find kortex_description)/arms/${arm}/${dof}dof/urdf/${arm}_macro.xacro" />
@@ -17,5 +17,11 @@
         <!-- Run the macros -->
         <!-- For gazebo and DART -->
-        <link name="world" />
+        <link name="world">
+            <inertial>
+                <origin xyz="0 0 0" rpy="0 0 0" />
+                <mass value="0"/>
+                <inertia ixx="0" ixy="0" ixz="0" iyy="0" iyz="0" izz="0" />
+            </inertial>
+        </link>
         <joint name="world_to_root" type="fixed">
             <child link="${prefix}base_link" />
@@ -54,14 +60,15 @@
             <xacro:load_forque parent="${prefix}${last_arm_link}"  prefix="${prefix}"/>
         </xacro:unless>
-        <!-- Load the realsense_camera -->
-        <xacro:unless value="${not realsense_cam}">
+        <!-- Load the feeding utensil -->
+        <xacro:unless value="${not feeding_utensil}">
             <!-- last_arm_link is defined in "$(find kortex_description)/arms/${arm}/urdf/${arm}_macro.xacro" -->
-            <xacro:include filename="$(find kortex_description)/tools/realsense_cam/realsense_cam_mount.xacro" />
-            <xacro:load_realsense_cam parent="${prefix}${last_arm_link}"  prefix="${prefix}" reflect="1"/>
+            <xacro:include filename="$(find kortex_description)/tools/feeding_utensil/feeding_utensil.xacro" />
+            <xacro:load_feeding_utensil parent="${prefix}finger_tip"  prefix="${prefix}"/>
         </xacro:unless>
-        <xacro:unless value="${not reflect_cam}">
+        <!-- Load the drinking utensil -->
+        <xacro:unless value="${not drinking_utensil}">
             <!-- last_arm_link is defined in "$(find kortex_description)/arms/${arm}/urdf/${arm}_macro.xacro" -->
-            <xacro:include filename="$(find kortex_description)/tools/realsense_cam/realsense_cam_mount.xacro" />
-            <xacro:load_realsense_cam parent="${prefix}${last_arm_link}"  prefix="${prefix}" reflect="-1"/>
+            <xacro:include filename="$(find kortex_description)/tools/drinking_utensil/drinking_utensil.xacro" />
+            <xacro:load_drinking_utensil parent="${prefix}finger_tip"  prefix="${prefix}"/>
         </xacro:unless>
         <!-- Load the Gazebo transmissions and gazebo_ros_control plugin -->

File: tools/forque/forque.xacro (robot description, xacro)
@@ -2,10 +2,11 @@
 <robot xmlns:xacro="http://ros.org/wiki/xacro">
   <xacro:macro name="load_forque" params="parent prefix">
-    <joint name="${prefix}forque_joint" type="fixed">
+    <joint name="${prefix}forque_tip_joint" type="fixed">
           <parent link="${parent}"/>
-          <child link="${prefix}forque"/>
-          <origin rpy="0.0 0.0 0" xyz="0.0 0.0 0.11"/>
+          <child link="${prefix}forque_tip"/>
+          <!-- <origin rpy="0.0 0.0 0" xyz="0.0 0.0 0.35"/> -->
+          <origin rpy="0.0 0.0 0" xyz="0.0 0.0 0.315"/>
     </joint>
-    <link name="${prefix}forque">
+    <link name="${prefix}forque_tip">
       <inertial>
           <origin xyz="0 0 0.091" rpy="0 0 0" />
@@ -16,5 +17,5 @@
         <origin xyz="0 0 0" rpy="0 0 0" />
         <geometry>
-          <mesh filename="package://kortex_description/tools/forque/forque.stl" scale="0.001 0.001 0.001"/>
+          <mesh filename="package://kortex_description/tools/forque/forque_tip.stl" scale="0.001 0.001 0.001"/>
         </geometry>
         <material name="carbon_fiber">
@@ -25,40 +26,8 @@
         <origin xyz="0 0 0" rpy="0 0 0" />
         <geometry>
-          <mesh filename="package://kortex_description/tools/forque/forque.stl" scale="0.001 0.001 0.001"/>
+          <mesh filename="package://kortex_description/tools/forque/forque_tip.stl" scale="0.001 0.001 0.001"/>
         </geometry>
       </collision>
     </link>
-    <gazebo reference="${prefix}forque">
-        <material>Gazebo/Black</material>
-    </gazebo>
-    <link name="${prefix}forque_end_effector">
-      <inertial>
-        <origin xyz="0 0 0" rpy="0 0 0" />
-        <mass value="0" />
-        <inertia ixx="0" ixy="0" ixz="0" iyy="0" iyz="0" izz="0" />
-      </inertial>
-    </link>
-    <joint name="${prefix}joint_forque_end_effector" type="fixed">
-      <parent link="${prefix}forque"/>
-      <child link="${prefix}forque_end_effector"/>
-      <axis xyz="0 0 0"/>
-      <limit effort="2000" lower="0" upper="0" velocity="1"/>
-      <origin rpy="0 0 0" xyz="0 0.007 0.18"/>
-    </joint>
-    <link name="${prefix}forque_tip">
-      <inertial>
-        <origin xyz="0 0 0" rpy="0 0 0" />
-        <mass value="0" />
-        <inertia ixx="0" ixy="0" ixz="0" iyy="0" iyz="0" izz="0" />
-      </inertial>
-    </link>
-    <joint name="${prefix}joint_forque_tip" type="fixed">
-      <parent link="${prefix}forque"/>
-      <child link="${prefix}forque_tip"/>
-      <axis xyz="0 0 0"/>
-      <limit effort="2000" lower="0" upper="0" velocity="1"/>
-      <!-- Rotation consistent with pointers of forque: -->
-      <origin rpy="-0.5 0 0" xyz="0.0 0.007 0.18"/>
-    </joint>
   </xacro:macro>
 </robot>
