Commit message: Mesh and Camera Calib for Realsense

File: grippers/robotiq_2f_85/urdf/robotiq_arg2f.xacro (robot description, xacro)
@@ -23,6 +23,6 @@
         <geometry>
           <!-- The DAE file doesn't show well in Gazebo so we're using the STL instead -->
-          <!-- <mesh filename="package://kortex_description/grippers/robotiq_2f_85/meshes/visual/robotiq_arg2f_85_base_link.dae" scale="0.001 0.001 0.001"/> -->
-          <mesh filename="package://kortex_description/grippers/robotiq_2f_85/meshes/collision/robotiq_arg2f_base_link.stl" />
+          <mesh filename="package://kortex_description/grippers/robotiq_2f_85/meshes/visual/robotiq_arg2f_85_base_link_realsense.dae" scale="0.001 0.001 0.001"/>
+          <!-- <mesh filename="package://kortex_description/grippers/robotiq_2f_85/meshes/collision/robotiq_arg2f_base_link.stl" /> -->
         </geometry>
         <material name="">
@@ -45,5 +45,5 @@
         <inertial>
             <origin xyz="0 0 0.058" rpy="0 0 0"/>
-            <mass value="0.925"/>
+            <mass value="0.97"/>
             <inertia ixx="0.000000" ixy="0.000000" ixz="0.000000" iyy="0.000000" iyz="0.000000" izz="0.000000"/>
         </inertial>

File: grippers/robotiq_2f_85/urdf/robotiq_arg2f_85_model_macro.xacro (robot description, xacro)
@@ -156,5 +156,5 @@
   </xacro:macro>
   <xacro:macro name="inner_knuckle_joint" params="prefix fingerprefix reflect">
-    <joint name="${prefix}${fingerprefix}_inner_knuckle_joint" type="fixed">
+    <joint name="${prefix}${fingerprefix}_inner_knuckle_joint" type="revolute">
       <!-- <origin xyz="0 ${reflect * -0.0127} 0.06142" rpy="${pi / 2 + .725} 0 ${(reflect - 1) * pi / 2}" /> -->
       <origin xyz="0 ${reflect * -0.0127} 0.06142" rpy="0 0 ${(1 + reflect) * pi / 2}"/>
@@ -167,5 +167,5 @@
   </xacro:macro>
   <xacro:macro name="inner_finger_joint" params="prefix fingerprefix">
-    <joint name="${prefix}${fingerprefix}_inner_finger_joint" type="fixed">
+    <joint name="${prefix}${fingerprefix}_inner_finger_joint" type="revolute">
       <origin xyz="0 0.0061 0.0471" rpy="0 0 0"/>
       <parent link="${prefix}${fingerprefix}_outer_finger" />
@@ -186,5 +186,5 @@
   <xacro:include filename="$(find kortex_description)/grippers/robotiq_2f_85/urdf/robotiq_arg2f.xacro" />
   <xacro:macro name="finger_joint" params="prefix">
-    <joint name="${prefix}finger_joint" type="fixed">
+    <joint name="${prefix}finger_joint" type="revolute">
       <origin xyz="0 -0.0306011 0.054904" rpy="0 0 ${pi}"/>
       <parent link="${prefix}robotiq_arg2f_base_link" />
@@ -196,5 +196,5 @@
   </xacro:macro>
   <xacro:macro name="right_outer_knuckle_joint" params="prefix">
-    <joint name="${prefix}right_outer_knuckle_joint" type="fixed">
+    <joint name="${prefix}right_outer_knuckle_joint" type="revolute">
       <origin xyz="0 0.0306011 0.054904" rpy="0 0 0"/>
       <parent link="${prefix}robotiq_arg2f_base_link" />

Commit message: cleanup + new utensil with F/T sensor

File: grippers/robotiq_2f_85/urdf/robotiq_arg2f.xacro (robot description, xacro)
@@ -59,5 +59,7 @@
         <parent link="${parent}" />
         <child link="${prefix}finger_tip" />
-        <origin xyz="0 0 0.163" rpy="0 0 0"/>
+        <!-- <origin xyz="0 0 0.163" rpy="0 0 0"/> -->
+        <origin xyz="0 0 0.17955" rpy="0 0 0"/>
+        <!-- Added 1.655mm because of the new finger tip -->
         <!-- <axis xyz="0 0 1" /> -->
     </joint>

File: tools/feeding_tool/feeding_tool.xacro (robot description, xacro)
@@ -142,5 +142,5 @@
       <!-- <origin rpy="0 0 0" xyz="0.095 0.007 0.0"/> -->
       <!-- <origin rpy="0 0 0" xyz="0.097 0.00 -0.002"/> -->
-      <origin rpy="0 0 0" xyz="0.1 -0.013 -0.002"/>
+      <origin rpy="0 0 0" xyz="0.13 0.0 0.0"/>
     </joint>
     <link name="${prefix}fork_tip">
