Commit message: tool mount/dismount in sim

File: robots/gen3_robotiq_2f_85.xacro (robot description, xacro)
@@ -6,10 +6,8 @@
     <xacro:arg name="vision" default="true" />
     <xacro:arg name="gripper" default="robotiq_2f_85" />
-    <xacro:arg name="forque" default="false" />
     <xacro:arg name="sim" default="false" />
     <xacro:arg name="prefix" default="" />
-    <xacro:arg name="feeding_utensil" default="false" />
-    <xacro:arg name="drinking_utensil" default="false" />
+    <xacro:arg name="tool" default="" />
     <xacro:include filename="$(find kortex_description)/robots/kortex_robot.xacro" />
-    <xacro:load_robot arm="$(arg arm)" gripper="$(arg gripper)" forque="$(arg forque)" feeding_utensil="$(arg feeding_utensil)" drinking_utensil="$(arg drinking_utensil)"  dof="$(arg dof)" vision="$(arg vision)" sim="$(arg sim)" prefix="$(arg prefix)" />
+    <xacro:load_robot arm="$(arg arm)" dof="$(arg dof)" vision="$(arg vision)" gripper="$(arg gripper)" sim="$(arg sim)" prefix="$(arg prefix)" tool="$(arg tool)"  />
 </robot>

File: robots/kortex_robot.xacro (robot description, xacro)
@@ -1,5 +1,5 @@
 <?xml version="1.0"?>
 <robot xmlns:xacro="http://ros.org/wiki/xacro">
-    <xacro:macro name="load_robot" params="arm gripper forque feeding_utensil drinking_utensil dof vision sim prefix">
+    <xacro:macro name="load_robot" params="arm dof vision gripper sim prefix tool">
         <!-- Files to include -->
         <xacro:include filename="$(find kortex_description)/arms/${arm}/${dof}dof/urdf/${arm}_macro.xacro" />
@@ -54,22 +54,28 @@
             </joint>
         </xacro:if>
-        <!-- Load the forque -->
-        <xacro:unless value="${not forque}">
-            <!-- last_arm_link is defined in "$(find kortex_description)/arms/${arm}/urdf/${arm}_macro.xacro" -->
-            <xacro:include filename="$(find kortex_description)/tools/forque/forque.xacro" />
-            <xacro:load_forque parent="${prefix}${last_arm_link}"  prefix="${prefix}"/>
-        </xacro:unless>
-        <!-- Load the feeding utensil -->
-        <xacro:unless value="${not feeding_utensil}">
-            <!-- last_arm_link is defined in "$(find kortex_description)/arms/${arm}/urdf/${arm}_macro.xacro" -->
-            <xacro:include filename="$(find kortex_description)/tools/feeding_utensil/feeding_utensil.xacro" />
-            <xacro:load_feeding_utensil parent="${prefix}finger_tip"  prefix="${prefix}"/>
-        </xacro:unless>
-        <!-- Load the drinking utensil -->
-        <xacro:unless value="${not drinking_utensil}">
-            <!-- last_arm_link is defined in "$(find kortex_description)/arms/${arm}/urdf/${arm}_macro.xacro" -->
-            <xacro:include filename="$(find kortex_description)/tools/drinking_utensil/drinking_utensil.xacro" />
-            <xacro:load_drinking_utensil parent="${prefix}finger_tip"  prefix="${prefix}"/>
-        </xacro:unless>
+        <!-- Load all tools -->
+        <xacro:if value="${tool == 'all'}">
+            <xacro:include filename="$(find kortex_description)/tools/feeding_tool/feeding_tool.xacro" />
+            <xacro:load_feeding_tool prefix="${prefix}"/>
+            <xacro:include filename="$(find kortex_description)/tools/drinking_tool/drinking_tool.xacro" />
+            <xacro:load_drinking_tool prefix="${prefix}"/>
+            <xacro:include filename="$(find kortex_description)/tools/wiping_tool/wiping_tool.xacro" />
+            <xacro:load_wiping_tool prefix="${prefix}"/>
+        </xacro:if>
+        <!-- Load the feeding tool -->
+        <xacro:if value="${tool == 'feeding'}">
+            <xacro:include filename="$(find kortex_description)/tools/feeding_tool/feeding_tool.xacro" />
+            <xacro:load_feeding_tool prefix="${prefix}"/>
+        </xacro:if>
+        <!-- Load the drinking tool -->
+        <xacro:if value="${tool == 'drinking'}">
+            <xacro:include filename="$(find kortex_description)/tools/drinking_tool/drinking_tool.xacro" />
+            <xacro:load_drinking_tool prefix="${prefix}"/>
+        </xacro:if>
+        <!-- Load the wiping tool -->
+        <xacro:if value="${tool == 'wiping'}">
+            <xacro:include filename="$(find kortex_description)/tools/drinking_tool/wiping_tool.xacro" />
+            <xacro:load_drinking_tool prefix="${prefix}"/>
+        </xacro:if>
         <!-- Load the Gazebo transmissions and gazebo_ros_control plugin -->
         <xacro:if value="${sim}">

File: tools/feeding_tool/feeding_tool.xacro (robot description, xacro)
@@ -1,9 +1,9 @@
 <?xml version="1.0" encoding="utf-8"?>
 <robot xmlns:xacro="http://ros.org/wiki/xacro">
-  <xacro:macro name="load_feeding_utensil" params="parent prefix">
-    <joint name="${prefix}feeding_utensil_joint" type="fixed">
-          <parent link="${parent}"/>
-          <child link="${prefix}forkbase"/>
-          <origin rpy="0.0 0.0 0.0" xyz="0.0 0.0 0.0"/>
+  <xacro:macro name="load_feeding_tool" params="prefix">
+    <joint name="finger_tip_to_forkbase" type="floating">
+        <parent link="finger_tip"/>
+        <child link="forkbase"/>
+        <origin xyz="0 0 0" rpy="0 0 0"/>
     </joint>
     <link name="${prefix}forkbase">
@@ -23,5 +23,5 @@
             <geometry>
                 <mesh
-                filename="package://kortex_description/tools/feeding_utensil/utensil_base.stl" />
+                filename="package://kortex_description/tools/feeding_tool/tool_base.stl" />
             </geometry>
             <material name="">
@@ -32,5 +32,5 @@
                 <origin xyz="0 0 0" rpy="0 0 0" />
             <geometry>
-                <mesh filename="package://kortex_description/tools/feeding_utensil/utensil_base.stl" />
+                <mesh filename="package://kortex_description/tools/feeding_tool/tool_base.stl" />
             </geometry>
         </collision>
@@ -52,5 +52,5 @@
             <geometry>
                 <mesh
-                filename="package://kortex_description/tools/feeding_utensil/utensil_roll.stl" />
+                filename="package://kortex_description/tools/feeding_tool/tool_pitch.stl" />
             </geometry>
             <material name="">
@@ -61,5 +61,5 @@
                 <origin xyz="0 0 0" rpy="0 0 0" />
             <geometry>
-                <mesh filename="package://kortex_description/tools/feeding_utensil/utensil_roll.stl" />
+                <mesh filename="package://kortex_description/tools/feeding_tool/tool_pitch.stl" />
             </geometry>
         </collision>
@@ -94,5 +94,5 @@
         <geometry>
             <mesh
-            filename="package://kortex_description/tools/feeding_utensil/roll_link_new2.stl" />
+            filename="package://kortex_description/tools/feeding_tool/tool_roll.stl" />
         </geometry>
         <material
@@ -108,5 +108,5 @@
         <geometry>
             <mesh
-            filename="package://kortex_description/tools/feeding_utensil/roll_link_new2.stl" />
+            filename="package://kortex_description/tools/feeding_tool/tool_roll.stl" />
         </geometry>
         </collision>
@@ -128,5 +128,5 @@
         velocity="8.4" />
     </joint>
-    <link name="${prefix}feeding_utensil_tip">
+    <link name="${prefix}feeding_tool_tip">
       <inertial>
         <origin xyz="0 0 0" rpy="0 0 0" />
@@ -135,7 +135,7 @@
       </inertial>
     </link>
-    <joint name="${prefix}joint_feeding_utensil_tip" type="fixed">
+    <joint name="${prefix}joint_feeding_tool_tip" type="fixed">
       <parent link="${prefix}forkroll"/>
-      <child link="${prefix}feeding_utensil_tip"/>
+      <child link="${prefix}feeding_tool_tip"/>
       <axis xyz="0 0 0"/>
       <limit effort="2000" lower="0" upper="0" velocity="1"/>
@@ -152,5 +152,5 @@
     </link>
     <joint name="${prefix}joint_fork_tip" type="fixed">
-      <parent link="${prefix}feeding_utensil_tip"/>
+      <parent link="${prefix}feeding_tool_tip"/>
       <child link="${prefix}fork_tip"/>
       <axis xyz="0 0 0"/>

File: tools/wiping_tool/wiping_tool.xacro (robot description, xacro)
@@ -1,11 +1,11 @@
 <?xml version="1.0" encoding="utf-8"?>
 <robot xmlns:xacro="http://ros.org/wiki/xacro">
-  <xacro:macro name="load_drinking_utensil" params="parent prefix">
-    <joint name="${prefix}drinking_utensil_joint" type="fixed">
-          <parent link="${parent}"/>
-          <child link="${prefix}drinkbase"/>
-          <origin rpy="0.0 0.0 0.0" xyz="0.0 0.0 0.0"/>
+  <xacro:macro name="load_wiping_tool" params="prefix">
+    <joint name="finger_tip_to_wipebase" type="floating">
+        <parent link="finger_tip"/>
+        <child link="wipebase"/>
+        <origin xyz="0 0 0" rpy="0 0 0"/>
     </joint>
-    <link name="${prefix}drinkbase">
+    <link name="${prefix}wipebase">
         <inertial>
             <origin xyz="0 0 0" rpy="0 0 0" />
@@ -23,5 +23,5 @@
             <geometry>
                 <mesh
-                filename="package://kortex_description/tools/drinking_utensil/utensil_base.stl" />
+                filename="package://kortex_description/tools/wiping_tool/tool_base.stl" />
             </geometry>
             <material name="">
@@ -32,9 +32,9 @@
                 <origin xyz="0 0 0" rpy="0 0 0" />
             <geometry>
-                <mesh filename="package://kortex_description/tools/drinking_utensil/utensil_base.stl" />
+                <mesh filename="package://kortex_description/tools/wiping_tool/tool_base.stl" />
             </geometry>
         </collision>
     </link>
-    <link name="${prefix}drink_tip">
+    <link name="${prefix}wipe_tip">
       <inertial>
         <origin xyz="0 0 0" rpy="0 0 0" />
@@ -43,7 +43,7 @@
       </inertial>
     </link>
-    <joint name="${prefix}joint_drink_tip" type="fixed">
-      <parent link="${prefix}drinkbase"/>
-      <child link="${prefix}drink_tip"/>
+    <joint name="${prefix}joint_wip_tip" type="fixed">
+      <parent link="${prefix}wipebase"/>
+      <child link="${prefix}wipe_tip"/>
       <axis xyz="0 0 0"/>
       <limit effort="2000" lower="0" upper="0" velocity="1"/>

Commit message: calibrated wipe tip

File: robots/gen3_robotiq_2f_85.xacro (robot description, xacro)
@@ -3,10 +3,10 @@
     <!-- Arguments -->
     <xacro:arg name="arm" default="gen3" />
-    <xacro:arg name="dof" default="6" />
-    <xacro:arg name="vision" default="true" />
+    <xacro:arg name="dof" default="7" />
+    <xacro:arg name="vision" default="false" />
     <xacro:arg name="gripper" default="robotiq_2f_85" />
     <xacro:arg name="sim" default="false" />
     <xacro:arg name="prefix" default="" />
-    <xacro:arg name="tool" default="" />
+    <xacro:arg name="tool" default="feeding" />
     <xacro:include filename="$(find kortex_description)/robots/kortex_robot.xacro" />
     <xacro:load_robot arm="$(arg arm)" dof="$(arg dof)" vision="$(arg vision)" gripper="$(arg gripper)" sim="$(arg sim)" prefix="$(arg prefix)" tool="$(arg tool)"  />

File: tools/feeding_tool/feeding_tool.xacro (robot description, xacro)
@@ -142,5 +142,5 @@
       <!-- <origin rpy="0 0 0" xyz="0.095 0.007 0.0"/> -->
       <!-- <origin rpy="0 0 0" xyz="0.097 0.00 -0.002"/> -->
-      <origin rpy="0 0 0" xyz="0.13 0.0 0.0"/>
+      <origin rpy="0 0 0" xyz="0.13 0.0 0.003"/>
     </joint>
     <link name="${prefix}fork_tip">

File: tools/wiping_tool/wiping_tool.xacro (robot description, xacro)
@@ -50,5 +50,5 @@
       <!-- <origin rpy="0 0 0" xyz="0.095 0.007 0.0"/> -->
       <!-- <origin rpy="0 0 0" xyz="0.097 0.00 -0.002"/> -->
-      <origin rpy="0 1.570796 0" xyz="0.27 0.095 -0.045"/>
+      <origin rpy="0 1.570796 0" xyz="0.089 -0.015 -0.078"/>
     </joint>
   </xacro:macro>
