Commit message: added tool urdfs

File: robots/kortex_robot.xacro (robot description, xacro)
@@ -75,6 +75,6 @@
         <!-- Load the wiping tool -->
         <xacro:if value="${tool == 'wiping'}">
-            <xacro:include filename="$(find kortex_description)/tools/drinking_tool/wiping_tool.xacro" />
-            <xacro:load_drinking_tool prefix="${prefix}"/>
+            <xacro:include filename="$(find kortex_description)/tools/wiping_tool/wiping_tool.xacro" />
+            <xacro:load_wiping_tool prefix="${prefix}"/>
         </xacro:if>
         <!-- Load the Gazebo transmissions and gazebo_ros_control plugin -->

File: robots/robot_holding_fork.urdf (robot description, URDF)
Before this commit: robot gen3_robotiq_2f_85, 29 links, 28 joints
Links:
- removed link feeding_utensil_tip
- added link feeding_tool_tip, mass 0
- link forkbase: geometry collision mesh filename=package://kortex_description/tools/feeding_tool/tool_base.s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; visual mesh filename=package://kortex_description/tools/feeding_tool/tool_base.s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
- link forkpitch: geometry collision mesh filename=package://kortex_description/tools/feeding_tool/tool_pitch.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; visual mesh filename=package://kortex_description/tools/feeding_tool/tool_pitch.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
- link forkroll: geometry collision mesh filename=package://kortex_description/tools/feeding_tool/tool_roll.s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; visual mesh filename=package://kortex_description/tools/feeding_tool/tool_roll.s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
Joints:
- removed joint feeding_utensil_joint
- removed joint joint_feeding_utensil_tip
- added joint finger_tip_to_forkbase: type floating, parent finger_tip, child forkbase, origin xyz=0 0 0 rpy=0 0 0
- added joint joint_feeding_tool_tip: type fixed, parent forkroll, child feeding_tool_tip, origin xyz=0.13 0.0 0.003 rpy=0 0 0, axis 0 0 0, limit lower=0 upper=0 effort=2000 velocity=1
- joint finger_tip_joint: origin xyz=0 0 0.163 rpy=0 0 0 -> xyz=0 0 0.17955 rpy=0 0 0
- joint joint_fork_tip: parent feeding_utensil_tip -> feeding_tool_tip

File: robots/robot_holding_wipe.urdf (robot description, URDF)
Before this commit: robot gen3_robotiq_2f_85, 26 links, 25 joints
Links:
- removed link drink_tip
- removed link drinkbase
- added link wipe_tip, mass 0
- added link wipebase, mass 0.072775; collision mesh filename=package://kortex_description/tools/wiping_tool/tool_base.stl; visual mesh filename=package://kortex_description/tools/wiping_tool/tool_base.stl
Joints:
- removed joint finger_tip_to_drinkbase
- removed joint joint_drink_tip
- added joint finger_tip_to_wipebase: type floating, parent finger_tip, child wipebase, origin xyz=0 0 0 rpy=0 0 0
- added joint joint_wip_tip: type fixed, parent wipebase, child wipe_tip, origin xyz=0.089 -0.015 -0.078 rpy=0 1.570796 0, axis 0 0 0, limit lower=0 upper=0 effort=2000 velocity=1
