Commit message: FEAST updates

File: robots/robot_holding_wipe.urdf (robot description, URDF)
Before this commit: robot gen3_robotiq_2f_85, 26 links, 25 joints
Joints:
- joint joint_wip_tip: origin xyz=0.089 -0.015 -0.078 rpy=0 1.570796 0 -> xyz=0.139 -0.015 -0.078 rpy=0 1.570796 0

File: tools/drinking_tool/drinking_tool.xacro (robot description, xacro)
@@ -50,5 +50,6 @@
       <!-- <origin rpy="0 0 0" xyz="0.095 0.007 0.0"/> -->
       <!-- <origin rpy="0 0 0" xyz="0.097 0.00 -0.002"/> -->
-      <origin rpy="0 1.570796 0" xyz="0.27 0.095 -0.045"/>
+      <!-- <origin rpy="0 1.570796 0" xyz="0.27 0.095 -0.045"/> -->
+      <origin rpy="0 1.570796 0" xyz="0.21 0.07 -0.037"/>
     </joint>
   </xacro:macro>

File: tools/wiping_tool/wiping_tool.xacro (robot description, xacro)
@@ -50,5 +50,5 @@
       <!-- <origin rpy="0 0 0" xyz="0.095 0.007 0.0"/> -->
       <!-- <origin rpy="0 0 0" xyz="0.097 0.00 -0.002"/> -->
-      <origin rpy="0 1.570796 0" xyz="0.089 -0.015 -0.078"/>
+      <origin rpy="0 1.570796 0" xyz="0.139 -0.015 -0.078"/>
     </joint>
   </xacro:macro>
